Commit message: fix(sim): correct RGB-D and IMU frame orientation

File: ubot_description/urdf/gazebo/ubot_gazebo.urdf.xacro (robot description, xacro)
@@ -78,4 +78,82 @@
             </sensor>
         </gazebo>
+        <!-- IMU SENSOR (MPU 9250 simulation) -->
+        <gazebo reference="${prefix}imu_link">
+            <sensor name="${prefix}imu_sensor" type="imu">
+                <topic>/imu</topic>
+                <update_rate>100</update_rate>
+                <always_on>1</always_on>
+                <visualize>false</visualize>
+                <imu>
+                    <!-- Angular velocity (gyroscope) -->
+                    <angular_velocity>
+                        <x>
+                            <noise type="gaussian">
+                                <mean>0.0</mean>
+                                <stddev>0.009</stddev>
+                                <bias_mean>0.00075</bias_mean>
+                                <bias_stddev>0.005</bias_stddev>
+                                <dynamic_bias_stddev>0.00002</dynamic_bias_stddev>
+                                <dynamic_bias_correlation_time>400.0</dynamic_bias_correlation_time>
+                            </noise>
+                        </x>
+                        <y>
+                            <noise type="gaussian">
+                                <mean>0.0</mean>
+                                <stddev>0.009</stddev>
+                                <bias_mean>0.00075</bias_mean>
+                                <bias_stddev>0.005</bias_stddev>
+                                <dynamic_bias_stddev>0.00002</dynamic_bias_stddev>
+                                <dynamic_bias_correlation_time>400.0</dynamic_bias_correlation_time>
+                            </noise>
+                        </y>
+                        <z>
+                            <noise type="gaussian">
+                                <mean>0.0</mean>
+                                <stddev>0.009</stddev>
+                                <bias_mean>0.00075</bias_mean>
+                                <bias_stddev>0.005</bias_stddev>
+                                <dynamic_bias_stddev>0.00002</dynamic_bias_stddev>
+                                <dynamic_bias_correlation_time>400.0</dynamic_bias_correlation_time>
+                            </noise>
+                        </z>
+                    </angular_velocity>
+                    <!-- Linear acceleration (accelerometer) -->
+                    <linear_acceleration>
+                        <x>
+                            <noise type="gaussian">
+                                <mean>0.0</mean>
+                                <stddev>0.017</stddev>
+                                <bias_mean>0.1</bias_mean>
+                                <bias_stddev>0.001</bias_stddev>
+                                <dynamic_bias_stddev>0.0002</dynamic_bias_stddev>
+                                <dynamic_bias_correlation_time>300.0</dynamic_bias_correlation_time>
+                            </noise>
+                        </x>
+                        <y>
+                            <noise type="gaussian">
+                                <mean>0.0</mean>
+                                <stddev>0.017</stddev>
+                                <bias_mean>0.1</bias_mean>
+                                <bias_stddev>0.001</bias_stddev>
+                                <dynamic_bias_stddev>0.0002</dynamic_bias_stddev>
+                                <dynamic_bias_correlation_time>300.0</dynamic_bias_correlation_time>
+                            </noise>
+                        </y>
+                        <z>
+                            <noise type="gaussian">
+                                <mean>0.0</mean>
+                                <stddev>0.017</stddev>
+                                <bias_mean>0.1</bias_mean>
+                                <bias_stddev>0.001</bias_stddev>
+                                <dynamic_bias_stddev>0.0002</dynamic_bias_stddev>
+                                <dynamic_bias_correlation_time>300.0</dynamic_bias_correlation_time>
+                            </noise>
+                        </z>
+                    </linear_acceleration>
+                </imu>
+                <gz_frame_id>${prefix}imu_link</gz_frame_id>
+            </sensor>
+        </gazebo>
         <xacro:macro name="wheel_gazebo" params="wheel_name">
             <gazebo reference="${prefix}${wheel_name}_link">

File: ubot_description/urdf/sensors/ubot_camera.urdf.xacro (robot description, xacro)
@@ -4,6 +4,6 @@
   <!-- Camera Physical Properties -->
   <xacro:property name="camera_mass" value="0.10321" />
-  <xacro:property name="camera_length" value="0.090" />  <!-- Typical depth camera length -->
-  <xacro:property name="camera_width" value="0.025" />
+  <xacro:property name="camera_width" value="0.090" />  <!-- Typical depth camera length -->
+  <xacro:property name="camera_length" value="0.025" />
   <xacro:property name="camera_height" value="0.025" />
   <!-- Center of Mass -->
@@ -18,4 +18,10 @@
     <!--CAMERA_LINK (Main camera body)-->
     <link name="${prefix}camera_link">
+      <!-- <visual>
+        <geometry>
+            <box size="${camera_length} ${camera_width} ${camera_height}"/>
+        </geometry>
+        <origin xyz="0 0 0" rpy="0 0 0"/>
+      </visual> -->
       <visual>
         <origin xyz="0 0 0" rpy="${pi/2} 0 ${pi/2}"/>
@@ -55,5 +61,5 @@
       <child link="${prefix}camera_depth_frame"/>
       <!-- Rotate to optical frame X right, Y down, Z forward -->
-      <origin xyz="0 0 0" rpy="${-pi/2} 0 ${-pi/2}"/>
+      <origin xyz="0 0 0" rpy="0 0 0"/>
     </joint>
     <!-- CAMERA_RGB_FRAME (Optical frame for RGB) Typically aligned with depth frame-->

File: ubot_description/urdf/sensors/ubot_imu.urdf.xacro (robot description, xacro)
@@ -10,5 +10,5 @@
   <xacro:property name="com_z" value="0.010541" />
   <xacro:property name="stand_height" value="${imu_height}" />
-  <xacro:property name="imu_x" value="0.2155" />
+  <xacro:property name="imu_x" value="0.0" />
   <xacro:property name="imu_y" value="0.0" />
   <xacro:property name="imu_z" value="-0.0075" />
