Commit message: feat(hw): implement and stabilize ros2_control hardware interface

File: ubot_description/urdf/body/ubot_wheel.urdf.xacro (robot description, xacro)
@@ -3,5 +3,5 @@
   <xacro:property name="wheel_radius" value="0.0325" />
   <xacro:property name="wheel_offset" value="0.0000" />
-  <xacro:property name="wheel_separation" value="0.2261" />
+  <xacro:property name="wheel_separation" value="0.255" />
   <xacro:property name="wheel_width" value="0.0264" />
   <xacro:property name="wheel_mass" value="0.4" />
@@ -13,8 +13,12 @@
     <link name="${prefix}front_left_wheel_link">
       <visual>
+        <!-- <geometry>
+            <mesh filename="package://ubot_description/meshes/wheel.stl" scale="0.001 0.001 0.001"/>
+        </geometry> -->
+        <!-- <origin xyz="0 0 0" rpy="0 0 ${-pi/2}"/> -->
+        <origin xyz="0 0 0" rpy="${pi/2} 0 0"/>
         <geometry>
-            <mesh filename="file://$(find ubot_description)/meshes/wheel.stl" scale="0.001 0.001 0.001"/>
+          <cylinder radius="${wheel_radius + wheel_offset}" length="${wheel_width}"/>
         </geometry>
-        <origin xyz="0 0 0" rpy="0 0 ${-pi/2}"/>
         <material name="dark_gray">
           <color rgba="0.2 0.2 0.2 1"/>
@@ -45,8 +49,12 @@
     <link name="${prefix}front_right_wheel_link">
       <visual>
+        <!-- <geometry>
+            <mesh filename="package://ubot_description/meshes/wheel.stl" scale="0.001 0.001 0.001"/>
+        </geometry>
+        <origin xyz="0 0 0" rpy="0 0 ${pi/2}"/> -->
+        <origin xyz="0 0 0" rpy="${pi/2} 0 0"/>
         <geometry>
-            <mesh filename="file://$(find ubot_description)/meshes/wheel.stl" scale="0.001 0.001 0.001"/>
+          <cylinder radius="${wheel_radius + wheel_offset}" length="${wheel_width}"/>
         </geometry>
-        <origin xyz="0 0 0" rpy="0 0 ${pi/2}"/>
         <material name="dark_gray">
           <color rgba="0.2 0.2 0.2 1"/>
@@ -76,8 +84,12 @@
     <link name="${prefix}rear_left_wheel_link">
       <visual>
+        <!-- <geometry>
+            <mesh filename="package://ubot_description/meshes/wheel.stl" scale="0.001 0.001 0.001"/>
+        </geometry>
+        <origin xyz="0 0 0" rpy="0 0 ${pi/2}"/> -->
+        <origin xyz="0 0 0" rpy="${pi/2} 0 0"/>
         <geometry>
-            <mesh filename="file://$(find ubot_description)/meshes/wheel.stl" scale="0.001 0.001 0.001"/>
+          <cylinder radius="${wheel_radius + wheel_offset}" length="${wheel_width}"/>
         </geometry>
-        <origin xyz="0 0 0" rpy="0 0 ${pi/2}"/>
         <material name="dark_gray">
           <color rgba="0.2 0.2 0.2 1"/>
@@ -99,6 +111,5 @@
       </inertial>
     </link>
-    <joint name="${prefix}rear_left_wheel_joint" type="continuous">
-      <axis xyz="0 1 0"/>
+    <joint name="${prefix}rear_left_wheel_joint" type="fixed">
       <parent link="${prefix}base_link"/>
       <child link="${prefix}rear_left_wheel_link"/>
@@ -107,8 +118,12 @@
     <link name="${prefix}rear_right_wheel_link">
       <visual>
+        <!-- <geometry>
+            <mesh filename="package://ubot_description/meshes/wheel.stl" scale="0.001 0.001 0.001"/>
+        </geometry>
+        <origin xyz="0 0 0" rpy="0 0 ${pi/2}"/> -->
+        <origin xyz="0 0 0" rpy="${pi/2} 0 0"/>
         <geometry>
-            <mesh filename="file://$(find ubot_description)/meshes/wheel.stl" scale="0.001 0.001 0.001"/>
+          <cylinder radius="${wheel_radius + wheel_offset}" length="${wheel_width}"/>
         </geometry>
-        <origin xyz="0 0 0" rpy="0 0 ${pi/2}"/>
         <material name="dark_gray">
           <color rgba="0.2 0.2 0.2 1"/>
@@ -130,6 +145,5 @@
       </inertial>
     </link>
-    <joint name="${prefix}rear_right_wheel_joint" type="continuous">
-      <axis xyz="0 1 0"/>
+    <joint name="${prefix}rear_right_wheel_joint" type="fixed">
       <parent link="${prefix}base_link"/>
       <child link="${prefix}rear_right_wheel_link"/>

File: ubot_description/urdf/ros2_control/ubot_ros2_control.xacro (robot description, xacro)
@@ -12,9 +12,9 @@
           <param name="left_wheel_name">front_left_wheel_joint</param>
           <param name="right_wheel_name">front_right_wheel_joint</param>
-          <param name="loop_rate">30</param>
+          <param name="loop_rate">20</param>
           <param name="device">/dev/ttyUSB0</param>
-          <param name="baud_rate">57600</param>
-          <param name="timeout_ms">1000</param>
-          <param name="enc_counts_per_rev">3000</param>
+          <param name="baud_rate">115200</param>
+          <param name="timeout_ms">2000</param>
+          <param name="enc_counts_per_rev">3650</param>
           <param name="pid_p">160</param>
           <param name="pid_d">30</param>
@@ -29,9 +29,9 @@
         <state_interface name="velocity"/>
       </joint>
-      <joint name="${prefix}rear_left_wheel_joint">
+      <!-- <joint name="${prefix}rear_left_wheel_joint">
         <command_interface name="velocity"/>
         <state_interface name="position"/>
         <state_interface name="velocity"/>
-      </joint>
+      </joint> -->
       <joint name="${prefix}front_right_wheel_joint">
         <command_interface name="velocity"/>
@@ -39,9 +39,9 @@
         <state_interface name="velocity"/>
       </joint>
-      <joint name="${prefix}rear_right_wheel_joint">
+      <!-- <joint name="${prefix}rear_right_wheel_joint">
         <command_interface name="velocity"/>
         <state_interface name="position"/>
         <state_interface name="velocity"/>
-      </joint>
+      </joint> -->
     </ros2_control>
   </xacro:macro>

Commit message: fix:sim_imu issue

File: ubot_description/urdf/body/ubot_wheel.urdf.xacro (robot description, xacro)
@@ -2,5 +2,5 @@
 <robot xmlns:xacro="http://www.ros.org/wiki/xacro">
   <xacro:property name="wheel_radius" value="0.033" />
-  <xacro:property name="wheel_separation" value="0.255" />
+  <xacro:property name="wheel_separation" value="0.264204" />  <!-- 2 * wheel_yoff = 2 * (base_width/2 + motor_cylinder_length) -->
   <xacro:property name="wheel_width" value="0.0264" />
   <xacro:property name="wheel_mass" value="0.4" />

File: ubot_description/urdf/gazebo/gazebo_control.xacro (robot description, xacro)
@@ -3,7 +3,9 @@
    <gazebo>
       <plugin filename="gz-sim-diff-drive-system" name="gz::sim::systems::DiffDrive">
-         <right_joint>right_wheel_joint</right_joint>
-         <left_joint>left_wheel_joint</left_joint>
-         <wheel_separation>0.134</wheel_separation>
+         <left_joint>front_left_wheel_joint</left_joint>
+         <left_joint>rear_left_wheel_joint</left_joint>
+         <right_joint>front_right_wheel_joint</right_joint>
+         <right_joint>rear_right_wheel_joint</right_joint>
+         <wheel_separation>${wheel_separation}</wheel_separation>
          <wheel_diameter>${2*wheel_radius}</wheel_diameter>
          <max_linear_acceleration>10</max_linear_acceleration>
@@ -17,6 +19,8 @@
       <plugin filename="gz-sim-joint-state-publisher-system" name="gz::sim::systems::JointStatePublisher">
          <topic>joint_states</topic>
-         <joint_name>right_wheel_joint</joint_name>
-         <joint_name>left_wheel_joint</joint_name>
+         <joint_name>front_left_wheel_joint</joint_name>
+         <joint_name>front_right_wheel_joint</joint_name>
+         <joint_name>rear_left_wheel_joint</joint_name>
+         <joint_name>rear_right_wheel_joint</joint_name>
       </plugin>
    </gazebo>

File: ubot_description/urdf/ros2_control/ubot_ros2_control.xacro (robot description, xacro)
@@ -10,8 +10,8 @@
           <plugin>ubot_control/UbotHardware</plugin>
           <!-- Only 2 "wheels" for control -->
-          <param name="left_wheel_name">front_left_wheel_joint</param>
-          <param name="right_wheel_name">front_right_wheel_joint</param>
-          <param name="right_wheel_name">rear_left_wheel_joint</param>
-          <param name="right_wheel_name">rear_right_wheel_joint</param>
+          <param name="front_left_wheel_name">front_left_wheel_joint</param>
+          <param name="front_right_wheel_name">front_right_wheel_joint</param>
+          <param name="rear_left_wheel_name">rear_left_wheel_joint</param>
+          <param name="rear_right_wheel_name">rear_right_wheel_joint</param>
           <param name="loop_rate">20</param>
           <param name="device">/dev/ttyUSB1</param>

File: ubot_description/urdf/sensors/ubot_camera.urdf.xacro (robot description, xacro)
@@ -3,5 +3,5 @@
   <xacro:property name="M_PI" value="3.1415926535897931" />
   <!-- Camera Physical Properties -->
-  <xacro:property name="camera_mass" value="0.10321" />
+  <xacro:property name="camera_mass" value="0.072" />  <!-- Intel RealSense D435 ~72 g -->
   <xacro:property name="camera_width" value="0.090" />  <!-- Typical depth camera length -->
   <xacro:property name="camera_length" value="0.025" />

File: ubot_description/urdf/sensors/ubot_imu.urdf.xacro (robot description, xacro)
@@ -2,5 +2,5 @@
 <robot xmlns:xacro="http://www.ros.org/wiki/xacro">
   <xacro:property name="M_PI" value="3.1415926535897931" />
-  <xacro:property name="imu_mass" value="0.10321" />
+  <xacro:property name="imu_mass" value="0.050" />  <!-- 9-DOF IMU module with PCB ~50 g -->
   <xacro:property name="imu_length" value="0.0259" />
   <xacro:property name="imu_width" value="0.0155" />
@@ -12,5 +12,5 @@
   <xacro:property name="imu_x" value="0.0" />
   <xacro:property name="imu_y" value="0.0" />
-  <xacro:property name="imu_z" value="-0.0075" />
+  <xacro:property name="imu_z" value="0.0" />
   <xacro:macro name="ubot_imu" params="prefix">
     <link name="${prefix}imu_link">
@@ -29,5 +29,5 @@
       <inertial>
           <origin xyz="${com_x} ${com_y} ${com_z}" rpy="0 0 0"/>
-          <mass value="${imu_mass*1.25}"/>
+          <mass value="${imu_mass}"/>
           <inertia ixx="${(1/12) * imu_mass * ((imu_width * imu_width) + (imu_height * imu_height))}"  ixy="0.0"  ixz="0.0"
                     iyy="${(1/12) * imu_mass * ((imu_length * imu_length) + (imu_height * imu_height))}"  iyz="0.0"

File: ubot_description/urdf/sensors/ubot_lidar.urdf.xacro (robot description, xacro)
@@ -2,5 +2,5 @@
 <robot xmlns:xacro="http://www.ros.org/wiki/xacro">
   <xacro:property name="M_PI" value="3.1415926535897931" />
-  <xacro:property name="lidar_mass" value="0.10321" />
+  <xacro:property name="lidar_mass" value="0.170" />  <!-- RPLIDAR A1/A2 ~170 g -->
   <xacro:property name="lidar_length" value="0.035" />
   <xacro:property name="lidar_width" value="0.035" />
@@ -35,8 +35,9 @@
       <inertial>
           <origin xyz="${com_x} ${com_y} ${com_z}" rpy="0 0 0"/>
-          <mass value="${lidar_mass*1.25}"/>
-          <inertia ixx="${(1/12) * lidar_mass * ((lidar_width * lidar_width) + (lidar_height * lidar_height))}"  ixy="0.0"  ixz="0.0"
-                    iyy="${(1/12) * lidar_mass * ((lidar_length * lidar_length) + (lidar_height * lidar_height))}"  iyz="0.0"
-                    izz="${(1/12) * lidar_mass * ((lidar_length * lidar_length) + (lidar_width * lidar_width))}"/>
+          <mass value="${lidar_mass}"/>
+          <!-- Cylinder inertia: r = lidar_width/2, h = lidar_height -->
+          <inertia ixx="${(1/12) * lidar_mass * (3*(lidar_width/2)*(lidar_width/2) + lidar_height*lidar_height)}"  ixy="0.0"  ixz="0.0"
+                    iyy="${(1/12) * lidar_mass * (3*(lidar_width/2)*(lidar_width/2) + lidar_height*lidar_height)}"  iyz="0.0"
+                    izz="${(1/2) * lidar_mass * (lidar_width/2)*(lidar_width/2)}"/>
       </inertial>
     </link>

File: ubot_description/urdf/sensors/ubot_ultrasonic.urdf.xacro (robot description, xacro)
@@ -2,5 +2,5 @@
 <robot xmlns:xacro="http://www.ros.org/wiki/xacro">
   <xacro:property name="M_PI" value="3.1415926535897931" />
-  <xacro:property name="ultrasonic_mass" value="0.010321" />
+  <xacro:property name="ultrasonic_mass" value="0.008" />  <!-- HC-SR04 module ~8 g -->
   <xacro:property name="ultrasonic_length" value="0.05" />
   <xacro:property name="ultrasonic_width" value="0.014" />
@@ -26,5 +26,5 @@
       <inertial>
           <origin xyz="${com_x} ${com_y} ${com_z}" rpy="0 0 0"/>
-          <mass value="${ultrasonic_mass*1.25}"/>
+          <mass value="${ultrasonic_mass}"/>
           <inertia ixx="${(1/12) * ultrasonic_mass * ((ultrasonic_width * ultrasonic_width) + (ultrasonic_height * ultrasonic_height))}"  ixy="0.0"  ixz="0.0"
                     iyy="${(1/12) * ultrasonic_mass * ((ultrasonic_length * ultrasonic_length) + (ultrasonic_height * ultrasonic_height))}"  iyz="0.0"
@@ -58,5 +58,5 @@
       <inertial>
           <origin xyz="${com_x} ${com_y} ${com_z}" rpy="0 0 0"/>
-          <mass value="${ultrasonic_mass*1.25}"/>
+          <mass value="${ultrasonic_mass}"/>
           <inertia ixx="${(1/12) * ultrasonic_mass * ((ultrasonic_width * ultrasonic_width) + (ultrasonic_height * ultrasonic_height))}"  ixy="0.0"  ixz="0.0"
                     iyy="${(1/12) * ultrasonic_mass * ((ultrasonic_length * ultrasonic_length) + (ultrasonic_height * ultrasonic_height))}"  iyz="0.0"
