Commit message: feat(nav): adjust robot description and sim launch for Nav2 bringup

File: ubot_description/urdf/body/ubot_base.urdf.xacro (robot description, xacro)
@@ -13,5 +13,5 @@
         <visual>
             <geometry>
-                <mesh filename="package://ubot_description/meshes/latest.stl" scale="1 1 1"/>
+                <mesh filename="file://$(find ubot_description)/meshes/latest.stl" scale="1 1 1"/>
             </geometry>
             <!-- <geometry>

File: ubot_description/urdf/body/ubot_wheel.urdf.xacro (robot description, xacro)
@@ -14,5 +14,5 @@
       <visual>
         <geometry>
-            <mesh filename="package://ubot_description/meshes/wheel.stl" scale="0.001 0.001 0.001"/>
+            <mesh filename="file://$(find ubot_description)/meshes/wheel.stl" scale="0.001 0.001 0.001"/>
         </geometry>
         <origin xyz="0 0 0" rpy="0 0 ${-pi/2}"/>
@@ -46,5 +46,5 @@
       <visual>
         <geometry>
-            <mesh filename="package://ubot_description/meshes/wheel.stl" scale="0.001 0.001 0.001"/>
+            <mesh filename="file://$(find ubot_description)/meshes/wheel.stl" scale="0.001 0.001 0.001"/>
         </geometry>
         <origin xyz="0 0 0" rpy="0 0 ${pi/2}"/>
@@ -77,5 +77,5 @@
       <visual>
         <geometry>
-            <mesh filename="package://ubot_description/meshes/wheel.stl" scale="0.001 0.001 0.001"/>
+            <mesh filename="file://$(find ubot_description)/meshes/wheel.stl" scale="0.001 0.001 0.001"/>
         </geometry>
         <origin xyz="0 0 0" rpy="0 0 ${pi/2}"/>
@@ -108,5 +108,5 @@
       <visual>
         <geometry>
-            <mesh filename="package://ubot_description/meshes/wheel.stl" scale="0.001 0.001 0.001"/>
+            <mesh filename="file://$(find ubot_description)/meshes/wheel.stl" scale="0.001 0.001 0.001"/>
         </geometry>
         <origin xyz="0 0 0" rpy="0 0 ${pi/2}"/>

File: ubot_description/urdf/sensors/ubot_camera.urdf.xacro (robot description, xacro)
@@ -27,5 +27,5 @@
         <origin xyz="0 0 0" rpy="${pi/2} 0 ${pi/2}"/>
         <geometry>
-          <mesh filename="package://ubot_description/meshes/camera.stl" scale="0.001 0.001 0.001"/>
+          <mesh filename="file://$(find ubot_description)/meshes/camera.stl" scale="0.001 0.001 0.001"/>
         </geometry>
         <material name="camera_black">
@@ -99,5 +99,5 @@
         <origin xyz="0 0 0" rpy="${pi/2} 0 ${pi/2}"/>
         <geometry>
-            <mesh filename="package://ubot_description/meshes/camera.stl" scale="0.001 0.001 0.001"/>
+            <mesh filename="file://$(find ubot_description)/meshes/camera.stl" scale="0.001 0.001 0.001"/>
         </geometry>
         <material name="white">

File: ubot_description/urdf/sensors/ubot_lidar.urdf.xacro (robot description, xacro)
@@ -18,5 +18,5 @@
         <origin xyz="0 0 0" rpy="0 0 0"/>
         <geometry>
-            <mesh filename="package://ubot_description/meshes/lidar.stl" scale="0.001 0.001 0.001"/>
+            <mesh filename="file://$(find ubot_description)/meshes/lidar.stl" scale="0.001 0.001 0.001"/>
         </geometry>
         <!-- <geometry>

File: ubot_description/urdf/sensors/ubot_ultrasonic.urdf.xacro (robot description, xacro)
@@ -18,5 +18,5 @@
         <origin xyz="-0.040 -0.057 0.019" rpy="0 0 ${pi}"/>
         <geometry>
-            <mesh filename="package://ubot_description/meshes/ultrasonic.stl" scale="0.001 0.001 0.001"/>
+            <mesh filename="file://$(find ubot_description)/meshes/ultrasonic.stl" scale="0.001 0.001 0.001"/>
         </geometry>
         <material name="white">
@@ -41,5 +41,5 @@
         <origin xyz="0.040 0.057 0.019" rpy="0 0 0"/>
         <geometry>
-            <mesh filename="package://ubot_description/meshes/ultrasonic.stl" scale="0.001 0.001 0.001"/>
+            <mesh filename="file://$(find ubot_description)/meshes/ultrasonic.stl" scale="0.001 0.001 0.001"/>
         </geometry>
         <!-- <geometry>

Commit message: Add platformio

File: ubot_description/urdf/body/ubot_base.urdf.xacro (robot description, xacro)
@@ -25,5 +25,5 @@
         <collision>
             <geometry>
-                <box size="${base_length} ${base_width} ${base_height}"/>
+                <box size="${base_length - 0.01} ${base_width - 0.01} ${base_height - 0.01}"/>
             </geometry>
             <origin xyz="0 0 ${base_height/2}" rpy="0 0 0"/>

File: ubot_description/urdf/gazebo/ubot_gazebo.urdf.xacro (robot description, xacro)
@@ -4,5 +4,5 @@
         <gazebo>
             <plugin filename="gz_ros2_control-system" name="gz_ros2_control::GazeboSimROS2ControlPlugin">
-            <parameters>$(find ubot_bringup)/config/ubot_controllers.yaml</parameters>
+            <parameters>$(find ubot_bringup)/config/sim_ubot_controllers.yaml</parameters>
             </plugin>
         </gazebo>

File: ubot_description/urdf/ros2_control/ubot_ros2_control.xacro (robot description, xacro)
@@ -6,30 +6,28 @@
         <xacro:if value="${use_gazebo}">
           <plugin>gz_ros2_control/GazeboSimSystem</plugin>
+          <joint name="${prefix}rear_left_wheel_joint">
+            <command_interface name="velocity"/>
+            <state_interface name="position"/>
+            <state_interface name="velocity"/>
+          </joint>
+          <joint name="${prefix}rear_right_wheel_joint">
+            <command_interface name="velocity"/>
+            <state_interface name="position"/>
+            <state_interface name="velocity"/>
+          </joint>
         </xacro:if>
         <xacro:unless value="${use_gazebo}">
           <plugin>ubot_control/UbotHardware</plugin>
-          <!-- Only 2 "wheels" for control -->
-          <param name="front_left_wheel_name">front_left_wheel_joint</param>
-          <param name="front_right_wheel_name">front_right_wheel_joint</param>
-          <param name="rear_left_wheel_name">rear_left_wheel_joint</param>
-          <param name="rear_right_wheel_name">rear_right_wheel_joint</param>
-          <param name="loop_rate">20</param>
-          <param name="device">/dev/ttyUSB1</param>
-          <param name="baud_rate">115200</param>
-          <param name="timeout_ms">2000</param>
-          <param name="enc_counts_per_rev">3650</param>
-          <param name="pid_p">160</param>
-          <param name="pid_d">30</param>
-          <param name="pid_i">15</param>
-          <param name="pid_o">50</param>
+          <param name="left_wheel_name">front_left_wheel_joint</param>
+          <param name="right_wheel_name">front_right_wheel_joint</param>
+          <param name="enc_counts_per_rev_left">3956</param>
+          <param name="enc_counts_per_rev_right">3956</param>
+          <param name="wheel_separation">0.264204</param>
+          <param name="wheel_radius">0.033</param>
+          <param name="loop_rate">30</param>
         </xacro:unless>
       </hardware>
-      <!-- Define all 4 wheel joints for visualization -->
+      <!-- Front wheels: velocity command + position/velocity state -->
       <joint name="${prefix}front_left_wheel_joint">
-        <command_interface name="velocity"/>
-        <state_interface name="position"/>
-        <state_interface name="velocity"/>
-      </joint>
-      <joint name="${prefix}rear_left_wheel_joint">
         <command_interface name="velocity"/>
         <state_interface name="position"/>
@@ -41,6 +39,17 @@
         <state_interface name="velocity"/>
       </joint>
+      <!-- Rear Wheels -->
+      <joint name="${prefix}rear_left_wheel_joint">
+        <!-- In Gazebo, we need command interfaces for the 4WD diff_drive_controller -->
+        <xacro:if value="${use_gazebo}">
+          <command_interface name="velocity"/>
+        </xacro:if>
+        <state_interface name="position"/>
+        <state_interface name="velocity"/>
+      </joint>
       <joint name="${prefix}rear_right_wheel_joint">
-        <command_interface name="velocity"/>
+        <xacro:if value="${use_gazebo}">
+          <command_interface name="velocity"/>
+        </xacro:if>
         <state_interface name="position"/>
         <state_interface name="velocity"/>
@@ -49,32 +58,2 @@
   </xacro:macro>
 </robot>
-<!-- <?xml version="1.0"?>
-<robot xmlns:xacro="http://www.ros.org/wiki/xacro">
-    <xacro:macro name="ubot_ros2_control" params="prefix use_gazebo">
-        <ros2_control name="UbotSystem" type="system">
-            <hardware>
-                <xacro:if value="${use_gazebo}">
-                    <plugin>gz_ros2_control/GazeboSimSystem</plugin>
-                </xacro:if>
-                <xacro:unless value="${use_gazebo}">
-                    <plugin>ubot_control/UbotHardwareInterface</plugin>
-                </xacro:unless>
-            </hardware>
-            <xacro:macro name="wheel_interfaces" params="name">
-                <joint name="${name}">
-                    <command_interface name="velocity">
-                        <param name="min">-10.0</param>
-                        <param name="max">10.0</param>
-                    </command_interface>
-                    <state_interface name="position"/>
-                    <state_interface name="velocity"/>
-                </joint>
-            </xacro:macro>
-            <xacro:wheel_interfaces name="${prefix}front_left_wheel_joint"/>
-            <xacro:wheel_interfaces name="${prefix}rear_left_wheel_joint"/>
-            <xacro:wheel_interfaces name="${prefix}front_right_wheel_joint"/>
-            <xacro:wheel_interfaces name="${prefix}rear_right_wheel_joint"/>
-        </ros2_control>
-    </xacro:macro>
-</robot>
- -->
