Commit message: feat(bench): low-cost indoor navigation benchmark (worlds, sensor models, harness, protocol)
New packages:
- ubot_worlds: Gazebo Harmonic worlds for the benchmark. arena_5x5 is a replica of the
  physical arena; small_house, bookstore and small_warehouse come from the AWS RoboMaker
  Harmonic ports (models fetched at a pinned commit, not committed). Conditions (glass,
  dynamic, degraded, low_light) are xacro args, and the glass/walker placements live in
  missions/<world>.yaml. It also holds ground-truth scan-plane and traversability maps and
  the generated missions.
- ubot_bench: datasheet sensor noise model (scan_model), Gazebo ground truth and collision
  episodes (gt_publisher), teleported multi-height ground-truth mapper (gt_map), mission
  generator, mapping (ground-truth pure pursuit + slam_toolbox) and navigation
  (AMCL + Nav2, ground-truth success) runners, an isolated/resumable experiment
  orchestrator, and the metrics/statistics/figures pipeline (evo, paired Wilcoxon + Holm,
  Cliff's delta, bootstrap CIs, McNemar, power). Research protocol in docs/PROTOCOL.md.

Changes to existing packages:
- ubot_description: sensor_profiles.yaml (REF/MS200/LD06/A1/OAK-D Lite from datasheets)
  drives the simulated LiDAR/depth sensor. Adds a bench bumper contact sensor,
  glass-transparent visibility masks and axle-aligned wheel friction. In sim the rear
  wheels are driven explicitly instead of via mimic joints.
- ubot_bringup: sim.launch.py takes world:=, condition:= and sensor_profile:=
  (default small_house); basic.sdf removed. The sim controller drives all four wheels.
- ubot_mono_nav: sim_mono.launch.py uses ubot_worlds.

Co-Authored-By: Claude Opus 5.5 <noreply@anthropic.com>

File: src/ubot/ubot_description/urdf/body/ubot_robot.urdf.xacro (robot description, xacro)
@@ -5,4 +5,8 @@
     <xacro:arg name="prefix" default=""/>
     <xacro:arg name="use_gazebo" default="false"/>
+    <!-- Simulated range sensor (ubot_description/config/sensor_profiles.yaml) and whether the
+         benchmark noise pipeline (ubot_bench scan_model) replaces Gazebo's own noise. -->
+    <xacro:arg name="sensor_profile" default="lidar_ms200"/>
+    <xacro:arg name="bench" default="false"/>
     <xacro:include filename="$(find ubot_description)/urdf/body/ubot_base.urdf.xacro"/>
     <xacro:include filename="$(find ubot_description)/urdf/sensors/ubot_lidar.urdf.xacro"/>
@@ -17,10 +21,10 @@
     <xacro:ubot_ros2_control prefix="$(arg prefix)" use_gazebo="$(arg use_gazebo)" />
     <xacro:if value="$(arg use_gazebo)">
-        <xacro:ubot_gazebo prefix="$(arg prefix)" />
+        <xacro:ubot_gazebo prefix="$(arg prefix)" sensor_profile="$(arg sensor_profile)" bench="$(arg bench)"/>
     </xacro:if>
     <xacro:ubot_base
     prefix="$(arg prefix)" />
     <xacro:ubot_wheel
-    prefix="$(arg prefix)" />
+    prefix="$(arg prefix)" rear_mimic="${'$(arg use_gazebo)' != 'true'}" />
     <xacro:ubot_lidar
     prefix="$(arg prefix)" />

File: src/ubot/ubot_description/urdf/body/ubot_wheel.urdf.xacro (robot description, xacro)
@@ -54,9 +54,17 @@
     </joint>
   </xacro:macro>
-  <xacro:macro name="ubot_wheel" params="prefix">
+  <!--
+    rear_mimic: true on the real robot (the ESP32 mirrors each front command to the rear motor;
+    the rear joints are mimic joints). In Gazebo it must be false: gz_ros2_control's mimic handling
+    only tracks the rear joint position and delivers no drive torque, so the rear wheels roll free,
+    the simulated robot is front-wheel drive, and an in-place turn pivots about the front axle
+    (0.25 m of base translation per 180 deg, measured). In simulation the rear wheels get their own
+    velocity command interfaces instead and the diff_drive_controller drives all four.
+  -->
+  <xacro:macro name="ubot_wheel" params="prefix rear_mimic:=true">
     <xacro:ubot_single_wheel prefix="${prefix}" name="front_left"  x_sign="1"  y_sign="1"  mesh="wheel_front_left"  mesh_x="0.28988" mesh_y="0.1132"/>
     <xacro:ubot_single_wheel prefix="${prefix}" name="front_right" x_sign="1"  y_sign="-1" mesh="wheel_front_right" mesh_x="0.28988" mesh_y="-0.1132"/>
-    <xacro:ubot_single_wheel prefix="${prefix}" name="rear_left"   x_sign="-1" y_sign="1"  mesh="wheel_rear_left"   mesh_x="0.03488" mesh_y="0.1132"  mimics="front_left_wheel_joint"/>
-    <xacro:ubot_single_wheel prefix="${prefix}" name="rear_right"  x_sign="-1" y_sign="-1" mesh="wheel_rear_right"  mesh_x="0.03488" mesh_y="-0.1132" mimics="front_right_wheel_joint"/>
+    <xacro:ubot_single_wheel prefix="${prefix}" name="rear_left"   x_sign="-1" y_sign="1"  mesh="wheel_rear_left"   mesh_x="0.03488" mesh_y="0.1132"  mimics="${'front_left_wheel_joint' if rear_mimic else ''}"/>
+    <xacro:ubot_single_wheel prefix="${prefix}" name="rear_right"  x_sign="-1" y_sign="-1" mesh="wheel_rear_right"  mesh_x="0.03488" mesh_y="-0.1132" mimics="${'front_right_wheel_joint' if rear_mimic else ''}"/>
   </xacro:macro>
 </robot>

File: src/ubot/ubot_description/urdf/gazebo/ubot_gazebo.urdf.xacro (robot description, xacro)
@@ -1,5 +1,5 @@
 <?xml version="1.0"?>
 <robot xmlns:xacro="http://www.ros.org/wiki/xacro">
-    <xacro:macro name="ubot_gazebo" params="prefix">
+    <xacro:macro name="ubot_gazebo" params="prefix sensor_profile:=lidar_ms200 bench:=false">
         <gazebo>
             <plugin filename="gz_ros2_control-system" name="gz_ros2_control::GazeboSimROS2ControlPlugin">
@@ -15,34 +15,71 @@
             </plugin>
         </gazebo>
-        <!-- FIXED LIDAR CONFIGURATION -->
+        <!--
+          2D range sensor, shaped by config/sensor_profiles.yaml[sensor_profile].
+          bench:=false  Gazebo applies constant Gaussian noise (gz_stddev) and publishes /scan
+                        (interactive sim.launch.py).
+          bench:=true   Gazebo publishes a clean scan on /scan_raw; ubot_bench's scan_model node
+                        applies the datasheet noise model and publishes /scan.
+          A depth-kind profile (OAK-D Lite) has no LiDAR at all; /scan comes from the depth image.
+          visibility_mask 0xFFFFFFFD hides visuals flagged 2 (glass in ubot_worlds), so the LiDAR
+          and depth camera see through glass as real ones largely do.
+        -->
+        <xacro:property name="bench_on" value="${str(bench).lower() in ('true', '1')}"/>
+        <xacro:property name="prof" value="${xacro.load_yaml('$(find ubot_description)/config/sensor_profiles.yaml')[sensor_profile]}"/>
+        <xacro:if value="${prof['kind'] == 'lidar'}">
         <gazebo reference="${prefix}lidar_link">
             <sensor name="${prefix}lidar_sensor" type="gpu_lidar">
-                <topic>/scan</topic>
-                <update_rate>10</update_rate>
+                <topic>${'/scan_raw' if bench_on else '/scan'}</topic>
+                <update_rate>${prof['rate_hz']}</update_rate>
                 <always_on>true</always_on>
-                <visualize>true</visualize>
+                <visualize>${'false' if bench_on else 'true'}</visualize>
                 <lidar>
                     <scan>
                         <horizontal>
-                            <samples>720</samples>
+                            <samples>${prof['samples']}</samples>
                             <resolution>1</resolution>
-                            <min_angle>-3.14159</min_angle>
-                            <max_angle>3.14159</max_angle>
+                            <min_angle>${-radians(prof['fov_deg']) / 2 + (radians(prof['fov_deg']) / prof['samples'] / 2 if prof['fov_deg'] == 360.0 else 0.0)}</min_angle>
+                            <max_angle>${radians(prof['fov_deg']) / 2 - (radians(prof['fov_deg']) / prof['samples'] / 2 if prof['fov_deg'] == 360.0 else 0.0)}</max_angle>
                         </horizontal>
                     </scan>
                     <range>
-                        <min>0.2</min>
-                        <max>30.0</max>
-                        <resolution>0.01</resolution>
+                        <min>${prof['range_min']}</min>
+                        <max>${prof['range_max']}</max>
+                        <resolution>0.001</resolution>
                     </range>
+                    <xacro:unless value="${bench_on}">
                     <noise>
                         <type>gaussian</type>
                         <mean>0.0</mean>
-                        <stddev>0.01</stddev>
+                        <stddev>${prof['gz_stddev']}</stddev>
                     </noise>
+                    </xacro:unless>
+                    <visibility_mask>4294967293</visibility_mask>
                 </lidar>
                 <gz_frame_id>${prefix}lidar_link</gz_frame_id>
             </sensor>
         </gazebo>
+        </xacro:if>
+        <!--
+          Benchmark bumper: a contact sensor on every chassis collision (the wheels are excluded,
+          they touch the floor by design). URDF->SDF lumps base_link into base_footprint and
+          renames its collisions, hence the generated names below. Published on the gz topic
+          /bench/contacts; ubot_bench gt_publisher turns it into /ground_truth/contacts.
+        -->
+        <xacro:if value="${bench_on}">
+        <gazebo reference="${prefix}base_link">
+            <sensor name="${prefix}bumper" type="contact">
+                <always_on>true</always_on>
+                <update_rate>50</update_rate>
+                <topic>/bench/contacts</topic>
+                <contact>
+                    <collision>${prefix}base_footprint_fixed_joint_lump__base_link_collision</collision>
+                    <collision>${prefix}base_footprint_fixed_joint_lump__base_link_collision_1</collision>
+                    <collision>${prefix}base_footprint_fixed_joint_lump__base_link_collision_2</collision>
+                    <collision>${prefix}base_footprint_fixed_joint_lump__lidar_link_collision_3</collision>
+                </contact>
+            </sensor>
+        </gazebo>
+        </xacro:if>
         <!-- RGB-D CAMERA SENSOR - FIXED -->
         <gazebo reference="${prefix}camera_link">
@@ -70,8 +107,9 @@
                     <depth_camera>
                         <clip>
-                            <near>0.1</near>
-                            <far>10.0</far>
+                            <near>0.20</near>   <!-- OAK-D Lite MinZ, extended disparity -->
+                            <far>8.0</far>      <!-- OAK-D Lite ideal depth range -->
                         </clip>
                     </depth_camera>
+                    <visibility_mask>4294967293</visibility_mask>
                 </camera>
                 <gz_frame_id>${prefix}camera_depth_frame</gz_frame_id>
@@ -165,5 +203,10 @@
         <!--
           Skid-steer friction.
-          mu1 acts along fdir1 (the rolling direction, +X) and mu2 across it (sideways).
+          fdir1 is expressed in the collision frame, which spins with the wheel, so it must be
+          the one direction that does not rotate: the axle (collision +Z, the cylinder axis).
+          With fdir1 = 1 0 0 the high/low friction directions would swap as each wheel turns.
+          mu1 therefore acts ACROSS the tyre (sideways) and mu2 ALONG it (rolling).
+          (The front-axle pivot of in-place turns is load distribution, not friction direction:
+          see ubot_wheel.urdf.xacro.)
           A 4-wheel skid-steer can only turn by scrubbing its tyres sideways, so mu2 MUST
           be low. With mu1 = mu2 = 1.1 the robot is effectively bolted to the floor: the
@@ -173,11 +216,11 @@
         <xacro:macro name="wheel_gazebo" params="wheel_name">
             <gazebo reference="${prefix}${wheel_name}_link">
-                <mu1>1.0</mu1>
-                <mu2>0.50</mu2>
+                <mu1>0.50</mu1>   <!-- sideways (along fdir1 = axle) -->
+                <mu2>1.0</mu2>    <!-- rolling direction -->
                 <kp>1000000.0</kp>
                 <kd>10.0</kd>
                 <minDepth>0.001</minDepth>
                 <maxVel>0.1</maxVel>
-                <fdir1>1 0 0</fdir1>
+                <fdir1>0 0 1</fdir1>
                 <material>Gazebo/Grey</material>
             </gazebo>

File: src/ubot/ubot_description/urdf/ros2_control/ubot_ros2_control.xacro (robot description, xacro)
@@ -6,6 +6,7 @@
     - The Gazebo sim plugin (gz_ros2_control/GazeboSimSystem)
   Drive configuration: 4WD, front-wheel encoders only.
-  Rear joints carry state interfaces only (no command interface on real hw).
-  In simulation all 4 joints carry command + state interfaces.
+  Real hardware: rear joints carry state interfaces only (the ESP32 mirrors the front command).
+  Simulation: all 4 joints carry command + state interfaces and the diff_drive_controller drives
+  all four (see ubot_wheel.urdf.xacro rear_mimic for why mimic joints do not work in Gazebo).
   IMPORTANT — joint structure rules:
     <joint> tags MUST be siblings of <hardware>, not children of it.
@@ -74,4 +75,7 @@
       -->
       <joint name="${prefix}rear_left_wheel_joint">
+        <xacro:if value="${use_gazebo}">
+          <command_interface name="velocity"/>
+        </xacro:if>
         <state_interface name="position"/>
         <state_interface name="velocity"/>
@@ -79,4 +83,7 @@
       <!-- Rear right — same as rear left -->
       <joint name="${prefix}rear_right_wheel_joint">
+        <xacro:if value="${use_gazebo}">
+          <command_interface name="velocity"/>
+        </xacro:if>
         <state_interface name="position"/>
         <state_interface name="velocity"/>
